File: DOCs/Designs/Tof180SensorBoard/Tof180Sensor.kicad_sch (KiCad schematic)
At the start: 6 parts, among them J1 Interface to P2, U1 VL53L5CX-SATEL, U2 VL53L5CX-SATEL, U3 VL53L5CX-SATEL, U4 VL53L5CX-SATEL, U5 PCF8575CTS/1,118

Commit message: Schematic Add pull-us to interrupt lines, now r1.0
Parts:
- added R1, R2, R3, R4, R5: 47k, symbol Device:R
Connections:
- net +3.3V: now also R1.1, R2.2, R3.2, R4.2, R5.2
- net INTb: now also R1.2
- net INTb_1: now also R2.1
- net INTb_2: now also R3.1
- net INTb_3: now also R4.1
- net INTb_4: now also R5.1
